File: Universal-Laser-Driver.kicad_pcb (KiCad board)
At the start: 2 copper layers, 16.5 x 9 mm, 15 parts, among them SW1 SW_SPST, U1 LTC3129IUD, U2 AD8515

Commit message: Updated to KiCAD 6
Other:
- net class Default removed
- net class Power removed
